File: chess_electronics/Chess_Electronics.kicad_sch (KiCad schematic)
At the start: 84 parts, among them J1 Screw_Terminal_01x16, J2 Screw_Terminal_01x16, J3 Screw_Terminal_01x16, J4 Screw_Terminal_01x16, J5 Screw_Terminal_01x16, J6 Screw_Terminal_01x16, J7 Screw_Terminal_01x16, J8 Screw_Terminal_01x16, J9 Barrel_Jack, U1 SN74LV4051AN, U2 SN74LV4051AN, U3 SN74LV4051AN, U4 SN74LV4051AN, U5 SN74LV4051AN, U6 SN74LV4051AN, U7 SN74LV4051AN, U8 SN74LV4051AN

Commit message: Update PCB to use two multiplexers by chaining signal and ground in opposite directions
Parts:
- removed C10, C11, C12, C13, C14, C15, C16, C17, C18, C19, C20, C21, C22, C23, C24, C25, C26, C27, C28, C29, C30, C31, C32, C33, C34, C35, C36, C37, C38, C39, C40, C41, C42, C43, C44, C45, C46, C47, C48, C49, C50, C51, C52, C53, C54, C55, C56, C57, C58, C59, C60, C61, C62, C63, C64, C65: C_Small_US, Capacitor_THT:C_Axial_L3.8mm_D2.6mm_P7.50mm_Horizontal, symbol Device:C_Small_US
- removed J1, J2, J3, J4, J5, J6, J7, J8: Screw_Terminal_01x16, KiCad:CUI_TB003-500-P16BE, symbol Connector:Screw_Terminal_01x16
- removed U3, U4, U5, U6, U7, U8: SN74LV4051AN, KiCad:N16, symbol 2025-09-05_00-43-07:SN74LV4051AN
- added J1, J2: Screw_Terminal_01x08, TerminalBlock:TerminalBlock_MaiXu_MX126-5.0-08P_1x08_P5.00mm, symbol Connector:Screw_Terminal_01x08
Connections:
- net A: no longer U2.11 (A)
- net B: no longer U2.10 (B)
- net C: no longer U2.9 (C)
- net Common: no longer U2.3 (COM)
- net GND: now also U2.3 (COM)
- net at U2.1 (Y4): now also J1.5 (Pin_5)
- net at C2.2: now also J2.1 (Pin_1)
- net at U2.14 (Y1): now also J1.2 (Pin_2)
- net at C4.2: now also J2.3 (Pin_3)
- net at U2.12 (Y3): now also J1.4 (Pin_4)
- net at U2.13 (Y0): now also J1.1 (Pin_1)
- net at U2.15 (Y2): now also J1.3 (Pin_3)
- net at U2.2 (Y6): now also J1.8 (Pin_8)
- net at U2.4 (Y7): now also J1.7 (Pin_7)
- net at U2.5 (Y5): now also J1.6 (Pin_6)
- net at C7.2: now also J2.6 (Pin_6)
- net at C8.2: now also J2.7 (Pin_7)
- net at C9.2: now also J2.8 (Pin_8)
- net at C3.2: now also J2.2 (Pin_2)
- net at C5.2: now also J2.4 (Pin_4)
- net at C6.2: now also J2.5 (Pin_5)
- net Mux1 INH: no longer names the net of U1.6 (INH)
- net Mux1 INH: no longer ESP32.30 (Pin_30)
- net Mux2 INH: no longer names the net of U2.6 (INH)
- net Mux2 INH: no longer ESP32.29 (Pin_29)
- net Mux3 INH renamed F
- net F: now also U2.9 (C)
- net Mux4 INH: no longer names the net of ESP32.27 (Pin_27)
- net Mux5 INH: no longer names the net of ESP32.26 (Pin_26)
- net Mux6 INH: no longer names the net of ESP32.25 (Pin_25)
- net Mux7 INH: no longer names the net of ESP32.24 (Pin_24)
- net Mux8 INH: no longer names the net of ESP32.23 (Pin_23)
- new net D: ESP32.30 (Pin_30), U2.11 (A)
- new net E: ESP32.29 (Pin_29), U2.10 (B)
